Commit message: update tau_ext inference

File: urdf/nero/nero_with_gripper.urdf (robot description, URDF)
Before this commit: robot nero, 14 links, 13 joints
Links:
- added link gripper_tcp
Joints:
- added joint gripper_tcp_joint: type fixed, parent gripper_base, child gripper_tcp, origin xyz=0 0 0.2145 rpy=0 0 0
